File: hardware/riscv/riscv.kicad_pcb (KiCad board)
At the start: 4 copper layers, 99 parts, among them IC1 MT28EW256ABA1HPC-0SIT, IC2 TPS562231DRLR, IC3 MAX3059ASA+T, IC4 LM5156HPWPR, IC5 TSZ124IYPT, J1 USB_B, J2 Conn_01x07, J3 Conn_01x02, J4 Conn_01x02, J5 Conn_01x03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

Commit message: sch should be fine now
Parts:
- added C1: 10nF, Capacitors_SMD:C_0805, F.Cu at (161.0, 74.5)
- added C37: 10nF, Capacitors_SMD:C_0805, F.Cu at (156.4, 73.6)
- added C38: 10nF, Capacitors_SMD:C_0805, F.Cu at (151.9, 73.6)
- added C39: 1uF, Capacitors_SMD:C_0805, F.Cu at (161.0, 71.7)
- added C40: 10uF, Capacitors_SMD:C_0805, F.Cu at (165.6, 71.7)
- added J10: Conn_01x03, Robohub:DG_PB_3, F.Cu at (152.7, 41.1)
- added J11: Conn_01x02, Robohub:DG235-5.0-02P, F.Cu at (152.7, 61.3)
- added J12: Conn_01x02, Robohub:DG235-5.0-02P, F.Cu at (175.4, 61.3)
- added J13: Conn_01x02, Robohub:DG235-5.0-02P, F.Cu at (164.1, 61.3)
- added J14: Conn_01x03, Robohub:DG_PB_3, F.Cu at (169.1, 41.1)
- added J8: Conn_01x20, Pin_Headers:Pin_Header_Straight_1x20_Pitch2.54mm, F.Cu at (125.5, 46.5)
- added J9: Conn_01x20, Pin_Headers:Pin_Header_Straight_1x20_Pitch2.54mm, F.Cu at (40.5, 46.5)
- added Q4: TK110P10PL,RQ, samac:TJ15P04M3RQS, F.Cu at (183.0, 120.5)
- added Q5: TK110P10PL,RQ, samac:TJ15P04M3RQS, F.Cu at (184.5, 104.5)
- added R28: 5R, Resistors_SMD:R_0805, F.Cu at (151.7, 82.2)
- added R29: 5R, Resistors_SMD:R_0805, F.Cu at (155.8, 82.2)
- added R30: 330k, Resistors_SMD:R_0805, F.Cu at (151.7, 85.1)
- added R31: 330k, Resistors_SMD:R_0805, F.Cu at (168.2, 67.2)
- added R32: 330k, Resistors_SMD:R_0805, F.Cu at (185.6, 54.1)
- added R33: 330k, Resistors_SMD:R_0805, F.Cu at (155.8, 85.1)
- added R34: 220k, Resistors_SMD:R_0805, F.Cu at (164.2, 80.2)
- added R35: 330k, Resistors_SMD:R_0805, F.Cu at (160.0, 80.2)
- added R36: 220k, Resistors_SMD:R_0805, F.Cu at (164.2, 77.3)
- added R37: 10k, Resistors_SMD:R_0805, F.Cu at (169.9, 70.0)
- added R38: 10k, Resistors_SMD:R_0805, F.Cu at (150.4, 92.4)
- added R39: 5k, Resistors_SMD:R_0805, F.Cu at (185.6, 57.0)
- added R40: 1k, Resistors_SMD:R_0805, F.Cu at (203.9, 39.5)
- added R41: 1k, Resistors_SMD:R_0805, F.Cu at (169.9, 72.9)
- added R42: 100k, Resistors_SMD:R_0805, F.Cu at (160.0, 83.1)
- added R43: 100k, Resistors_SMD:R_0805, F.Cu at (189.8, 54.1)
- added R44: 50k, Resistors_SMD:R_0805, F.Cu at (155.8, 88.0)
- added R45: 10k, Resistors_SMD:R_0805, F.Cu at (151.7, 88.0)
- added R46: 10k, Resistors_SMD:R_0805, F.Cu at (174.1, 70.0)
- added R47: 5k, Resistors_SMD:R_0805, F.Cu at (172.4, 67.2)
- added R48: 100k, Resistors_SMD:R_0805, F.Cu at (168.3, 75.8)
- added R49: 100k, Resistors_SMD:R_0805, F.Cu at (185.6, 59.9)
- added R50: 50k, Resistors_SMD:R_0805, F.Cu at (154.6, 90.8)
- added R51: 100k, Resistors_SMD:R_0805, F.Cu at (189.8, 57.0)
- added R52: 100k, Resistors_SMD:R_0805, F.Cu at (160.0, 86.0)
- added R53: 10k, Resistors_SMD:R_0805, F.Cu at (203.9, 42.3)
- added R54: 10k, Resistors_SMD:R_0805, F.Cu at (208.0, 39.5)
- added R55: 10R, Resistors_SMD:R_0805, F.Cu at (168.3, 78.7)
- added R56: 10R, Resistors_SMD:R_0805, F.Cu at (176.5, 67.2)
- added U8: LM7332, Housings_SSOP:VSSOP-8_3.0x3.0mm_Pitch0.65mm, F.Cu at (149.5, 112.0)
- added U9: IR2104, Housings_SOIC:SOIC-8_3.9x4.9mm_Pitch1.27mm, F.Cu at (134.5, 104.0)
- D5: value BAT54S -> D_Schottky; footprint TO_SOT_Packages_SMD:SOT-23 -> Diodes_SMD:D_SMA
- R11: value 1M -> 330k
- R12, R13: value 100k -> 91k
- R14, R15: value 10k -> 240k
- moved R15 62.7 mm to (160.0, 77.3), turned to 0 degrees
- moved R14 59.2 mm to (155.8, 79.3), turned to 0 degrees
- moved R13 57.4 mm to (155.8, 76.4), turned to 0 degrees
- moved R12 51.3 mm to (151.7, 77.3), turned to 0 degrees
- moved D5 38.4 mm to (134.5, 99.0)
Connections:
- C29 pad 1: ADC_AC_400V -> Net-(C29-Pad1)
- D5 pad 1: FB_PGND -> Net-(C40-Pad1)
- D5 pad 2: +3V3 -> +12V
- FB1 pad 2: Net-(FB1-Pad2) -> VREF_FB
- IC5 pad 14: Net-(IC5-Pad14) -> ADC_X10
- IC5 pad 2: ADC_AC_400V -> Net-(C29-Pad1)
- IC5 pad 3: Net-(D5-Pad3) -> Net-(IC5-Pad3)
- IC5 pad 7: Net-(IC5-Pad7) -> ADC_TC_X50
- IC5 pad 8: Net-(IC5-Pad8) -> ADC_DIV10
- R12 pad 1: Net-(R12-Pad1) -> FB_PGND
- R12 pad 2: Net-(R11-Pad1) -> Net-(C1-Pad1)
- R13 pad 1: Net-(D5-Pad3) -> FB_PGND
- R13 pad 2: Net-(R12-Pad1) -> Net-(C37-Pad1)
- R14 pad 1: Net-(FB1-Pad2) -> Net-(C1-Pad1)
- R14 pad 2: Net-(D5-Pad3) -> Net-(C1-Pad2)
- R15 pad 1: Net-(D5-Pad3) -> Net-(C37-Pad1)
- R15 pad 2: FB_PGND -> Net-(C37-Pad2)
- U3 pad 16: Net-(U3-Pad16) -> ADC_TC_X50
- U3 pad 17: Net-(U3-Pad17) -> ADC_X10
- U3 pad 18: Net-(U3-Pad18) -> ADC_DIV10
- U3 pad 23: Net-(U3-Pad23) -> GPIO_PA0
- U3 pad 29: Net-(U3-Pad29) -> DACOUT0
- U3 pad 30: Net-(U3-Pad30) -> DACOUT1
- U3 pad 31: Net-(U3-Pad31) -> GPIO_PA6
- U3 pad 32: Net-(U3-Pad32) -> GPIO_PA7
- U3 pad 33: Net-(U3-Pad33) -> GPIO_PC4
- U3 pad 34: Net-(U3-Pad34) -> GPIO_PC5
- U3 pad 35: Net-(U3-Pad35) -> MOS_PP_PWM_IN_2
- U3 pad 36: Net-(U3-Pad36) -> GPIO_PB1
- U3 pad 37: Net-(U3-Pad37) -> FB_PGND
- U3 pad 53: Net-(U3-Pad53) -> GPIO_PB14
- U3 pad 54: Net-(U3-Pad54) -> GPIO_PB15
- U3 pad 63: Net-(U3-Pad63) -> GPIO_PC6
- U3 pad 67: Net-(U3-Pad67) -> GPIO_PA8
- U3 pad 69: Net-(U3-Pad69) -> GPIO_PA10
- U3 pad 78: Net-(U3-Pad78) -> GPIO_PC10
- U3 pad 79: Net-(U3-Pad79) -> GPIO_PC11
- U3 pad 80: Net-(U3-Pad80) -> GPIO_PC12
- U3 pad 83: Net-(U3-Pad83) -> GPIO_PD2
- U3 pad 84: Net-(U3-Pad84) -> GPIO_PD3
- U3 pad 87: Net-(U3-Pad87) -> GPIO_PD6
- U3 pad 88: Net-(U3-Pad88) -> GPIO_PD7
- U3 pad 91: Net-(U3-Pad91) -> GPIO_PB5
- U3 pad 92: Net-(U3-Pad92) -> GPIO_PB6
- U3 pad 95: Net-(U3-Pad95) -> GPIO_PB8
- U3 pad 96: Net-(U3-Pad96) -> GPIO_PB9
- U3 pad 97: Net-(U3-Pad97) -> GPIO_PE0
- U3 pad 98: Net-(U3-Pad98) -> GPIO_PE1
Routing:
- net Net-(IC5-Pad3): track 0.00 -> 13.7 mm
- net Net-(D5-Pad3): track 13.7 -> 0.00 mm
- net VREF_FB: track 0.00 -> 1.55 mm
- net Net-(FB1-Pad2): track 1.55 -> 0.00 mm

Commit message: rough positioning
Parts:
- Q4, Q5, R11, R30, R32, R34: moved to B.Cu
- moved J12 148.3 mm to (38.5, 118.5)
- moved R32 134.3 mm to (61.5, 105.5), turned to 270 degrees
- moved R39 128.9 mm to (65.0, 102.5), turned to 180 degrees
- moved J13 128.0 mm to (49.5, 118.5)
- moved J11 121.3 mm to (38.5, 102.0), turned to 270 degrees
- moved J10 118.1 mm to (43.5, 86.0), turned to 270 degrees
- moved C1 114.6 mm to (49.0, 98.8), turned to 90 degrees
- moved R31 110.4 mm to (65.5, 107.5)
- moved R13 108.4 mm to (48.0, 87.5)
- moved R29 108.1 mm to (48.0, 89.5), turned to 180 degrees
- moved R15 108.1 mm to (52.5, 88.2)
- moved C37 107.6 mm to (49.5, 85.2)
- moved R37 107.3 mm to (68.5, 105.0), turned to 90 degrees
- moved R14 105.7 mm to (51.8, 97.8)
- moved R36 105.2 mm to (62.0, 102.5), turned to 180 degrees
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Routing:
- net VREF: track 80.6 -> 32.1 mm
- net ADC_AC_400V: track 55.6 -> 11.1 mm, vias 2 -> 1
- net WS_DIN: track 47.8 -> 9.82 mm
- net VIN_MOS_PP_OUT_2: track 0.00 -> 15.5 mm
- net Net-(C37-Pad2): track 0.00 -> 14.1 mm
- net Net-(Q4-Pad1): track 0.00 -> 13.7 mm, vias 0 -> 1
- net Net-(J3-Pad1): track 13.0 -> 0.00 mm
- net Net-(J3-Pad2): track 12.8 -> 0.05 mm
- net Net-(C1-Pad2): track 0.00 -> 10.5 mm
- net Net-(IC3-Pad6): track 15.3 -> 5.00 mm
- net Net-(IC5-Pad3): track 13.7 -> 4.75 mm, vias 0 -> 1
- net Net-(IC3-Pad7): track 14.4 -> 5.82 mm
- net FB_PGND: track 249.2 -> 240.8 mm
- net Net-(C37-Pad1): track 0.00 -> 8.11 mm
- net +3V3: track 148.3 -> 140.7 mm
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