File: hardware/riscv/riscv.sch (KiCad schematic (older format))
At the start: 111 parts, among them IC1 MT28EW256ABA1HPC-0SIT, IC2 TPS562231DRLR, IC3 MAX3059ASA+T, IC4 LM5156HPWPR, IC5 TSZ124IYPT, J1 USB_B, J2 Conn_01x07, J3 Conn_01x02, J4 Conn_01x02, J5 Conn_01x03, J6 Conn_01x02, J7 Conn_01x02, Q1 TK110P10PL,RQ, Q2 TK110P10PL,RQ, Q3 STL4N10F7, SW1 SW_SPST, U1 USBLC6-2SC6, U2 LIS2DE12, U3 GD32VF103VBT6, U4 MAX485E, U5 NCP1117-3.3_TO252, U6 IR2104, U7 MCP1501, Y1 CSTCE8M00G52A

Commit message: sch should be fine now
Parts:
- added C1, C37: 10nF, Capacitors_SMD:C_0805, symbol Device:C
- added C39: 1uF, Capacitors_SMD:C_0805, symbol Device:C
- added C40: 10uF, Capacitors_SMD:C_0805, symbol Device:C
- added D5: D_Schottky, Diodes_SMD:D_SMA, symbol Device:D_Schottky
- added J10, J14: Conn_01x03, Robohub:DG_PB_3, symbol Connector_Generic:Conn_01x03
- added J12, J13: Conn_01x02, Robohub:DG235-5.0-02P, symbol Connector_Generic:Conn_01x02
- added J8, J9: Conn_01x20, Pin_Headers:Pin_Header_Straight_1x20_Pitch2.54mm, symbol Connector_Generic:Conn_01x20
- added Q4, Q5: TK110P10PL,RQ, samac:TJ15P04M3RQS, symbol samac:TK110P10PL,RQ
- added R12, R13: 91k, Resistors_SMD:R_0805, symbol Device:R
- added R14, R15: 240k, Resistors_SMD:R_0805, symbol Device:R
- added R28, R29: 5R, Resistors_SMD:R_0805, symbol Device:R
- added R45, R46, R53, R54: 10k, Resistors_SMD:R_0805, symbol Device:R
- added R47: 5k, Resistors_SMD:R_0805, symbol Device:R
- added R48, R49, R51, R52: 100k, Resistors_SMD:R_0805, symbol Device:R
- added R50: 50k, Resistors_SMD:R_0805, symbol Device:R
- added R55, R56: 10R, Resistors_SMD:R_0805, symbol Device:R
- added U8: LM7332, Housings_SSOP:VSSOP-8_3.0x3.0mm_Pitch0.65mm, symbol Amplifier_Operational:LM7332
- added U9: IR2104, Housings_SOIC:SOIC-8_3.9x4.9mm_Pitch1.27mm, symbol Driver_FET:IR2104
- gave numbers to parts that had none: 17
Connections:
- net +12V: now also C39.1, D5.2 (A), J8.19 (Pin_19), J9.19 (Pin_19), U8.8 (V+), U9.1 (VCC), U9.3 (~SD)
- net +3V3: now also J8.17 (Pin_17), J9.17 (Pin_17)
- net +5V: now also J8.18 (Pin_18), J9.18 (Pin_18)
- net GND: now also U3.37 (PB2/BOOT1), C39.2, J10.1 (Pin_1), J12.1 (Pin_1), J13.1 (Pin_1), J14.3 (Pin_3), J8.1 (Pin_1), J8.11 (Pin_11), J8.16 (Pin_16), J8.20 (Pin_20), J8.6 (Pin_6), J9.1 (Pin_1), J9.11 (Pin_11), J9.16 (Pin_16), J9.20 (Pin_20), J9.6 (Pin_6), Q5.3, R12.1, R13.1, R46.2, R49.2, R52.1, R54.1, U8.4 (V-), U9.4 (COM)
- net VREF_FB: now also R45.2, R48.2
- net ADC_X10: now reaches U3.17 (PC2/ADC1_IN12)
- net ADC_X10: now also IC5.14 (OUT4), R47.2
- net ADC_DIV10: now reaches U3.18 (PC3/ADC1_IN13)
- net ADC_DIV10: now also IC5.8 (OUT3), R50.2
- net GPIO_PA0: now reaches U3.23 (PA0/WKUP/USART1_CTS/ADC1_IN0/TIM1_CH0_ETI/TIM4_CH1)
- net GPIO_PA0: now also J9.2 (Pin_2)
- net DACOUT0: now reaches U3.29 (PA4/SPI0_NSS/USART1_CK/ADC1_IN4/DAC_OUT0)
- net DACOUT0: now also U8.3 (+)
- net DACOUT1: now reaches U3.30 (PA5/SPI0_SCK/ADC1_IN5/DAC_OUT1)
- net DACOUT1: now also U8.5 (+)
- net GPIO_PA6: now reaches U3.31 (PA6/SPI0_MISO/ADC1_IN6/TIM2_CH0)
- net GPIO_PA6: now also J9.3 (Pin_3)
- net GPIO_PA7: now reaches U3.32 (PA7/SPI0_MOSI/ADC1_IN7/TIM2_CH1)
- net GPIO_PA7: now also J9.4 (Pin_4)
- net GPIO_PC4: now reaches U3.33 (PC4/ADC1_IN14)
- net GPIO_PC4: now also J9.5 (Pin_5)
- net GPIO_PC5: now reaches U3.34 (PC5/ADC1_IN15)
- net GPIO_PC5: now also J9.7 (Pin_7)
- net MOS_PP_PWM_IN_2: now reaches U3.35 (PB0/ADC1_IN8/TIM2_CH2)
- net MOS_PP_PWM_IN_2: now also U9.2 (IN)
- net GPIO_PB1: now reaches U3.36 (PB1/ADC1_IN9/TIM2_CH3)
- net GPIO_PB1: now also J9.8 (Pin_8)
- net GPIO_PB14: now reaches U3.53 (PB14/SPI1_MISO/USART2_RTS/TIM0_CH1_ON)
- net GPIO_PB14: now also J8.14 (Pin_14)
- net GPIO_PB15: now reaches U3.54 (PB15/SPI1_MODI/TIM0_CH2_ON/I2S1_SD)
- net GPIO_PB15: now also J8.15 (Pin_15)
- net GPIO_PC6: now reaches U3.63 (PC6/I2S1_MCK)
- net GPIO_PC6: now also J8.13 (Pin_13)
- net GPIO_PA8: now reaches U3.67 (PA8/USART0_CK/TIM0_CH0/CK_OUT0/USBFS_SOF)
- net GPIO_PA8: now also J8.12 (Pin_12)
- net GPIO_PA10: now reaches U3.69 (PA10/USART0_RX/TIM0_CH2/USBFS_ID)
- net GPIO_PA10: now also J8.10 (Pin_10)
- net GPIO_PC10: now reaches U3.78 (PC10/USART3_TX)
- net GPIO_PC10: now also J8.9 (Pin_9)
- net GPIO_PC11: now reaches U3.79 (PC11/USART3_RX)
- net GPIO_PC11: now also J8.4 (Pin_4)
- net GPIO_PC12: now reaches U3.80 (PC12/UART4_TX)
- net GPIO_PC12: now also J8.5 (Pin_5)
- net GPIO_PD2: now reaches U3.83 (PD2/TIM2_ETI/UART4_RX)
- net GPIO_PD2: now also J8.7 (Pin_7)
- net GPIO_PD3: now reaches U3.84 (PD3)
- net GPIO_PD3: now also J8.8 (Pin_8)
- net GPIO_PD6: now reaches U3.87 (PD6/EXMC_NWAIT)
- net GPIO_PD6: now also J8.2 (Pin_2)
- net GPIO_PD7: now reaches U3.88 (PD7/EXMC_NE0)
- net GPIO_PD7: now also J8.3 (Pin_3)
- net GPIO_PB5: now reaches U3.91 (PB5/I2C0_SMBA/SPI2_MOSI/I2S2_SD)
- net GPIO_PB5: now also J9.14 (Pin_14)
- net GPIO_PB6: now reaches U3.92 (PB6/I2C0_SCL/TIM3_CH0)
- net GPIO_PB6: now also J9.15 (Pin_15)
- net GPIO_PB8: now reaches U3.95 (PB8/TIM3_CH2)
- net GPIO_PB8: now also J9.9 (Pin_9)
- net GPIO_PB9: now reaches U3.96 (PB9/TIM3_CH3)
- net GPIO_PB9: now also J9.10 (Pin_10)
- net GPIO_PE0: now reaches U3.97 (PE0/TIM3_ETI/EXMC_NBL0)
- net GPIO_PE0: now also J9.12 (Pin_12)
- net GPIO_PE1: now reaches U3.98 (PE1/EXMC_NBL1)
- net GPIO_PE1: now also J9.13 (Pin_13)
- net at IC5.10 (IN3+): now also R48.1, R49.1, R53.2
- net at IC5.12 (IN4+): now also R45.1, R46.1, R51.2
- net at IC5.13 (IN4-): now also R47.1, R52.2
- net at IC5.9 (IN3-): now also R50.1, R54.2
- new net: Q5.1, R56.1
- new net: Q4.1, R55.1
- new net: R55.2, U9.7 (HO)
- new net: R56.2, U9.5 (LO)
- new net: C40.1, D5.1 (K), U9.8 (VB)
- new net: C37.2, R15.2, R29.1, U8.1
- new net: C37.1, R13.2, R15.1, U8.2 (-)
- new net: C1.1, R12.2, R14.1, U8.6 (-)
- new net: C1.2, R14.2, R28.1, U8.7
- new net BUFFERED_DACOUT0: J10.2 (Pin_2), R29.2
- new net BUFFERED_DACOUT1: J10.3 (Pin_3), R28.2
- new net IN_ADC_DIV10: J13.2 (Pin_2), R53.1
- new net IN_ADC_X10: J12.2 (Pin_2), R51.1
- new net VIN_MOS_PP_2: J14.1 (Pin_1), Q4.2
- new net VIN_MOS_PP_OUT_2: C40.2, J14.2 (Pin_2), Q4.3, Q5.2, U9.6 (VS)
Other:
- note added: "12V to 5V buck"
- note added: "2X PWM Push-Pull"
- note added: "ADC IN\nx 0.1, center at VREF/2"
- note added: "ADC IN\nx10, center at VREF/2"
- note added: "CAN Transceiver"
- note added: "DAC Buffer +12V 100mA\nX2"
- note added: "RS485"
- note added: "USB + ESD"
- note added: "extra user GPIO"
- moved on the sheet: C12, C15, C25, C29, C38, D1, D2, D3, FB1, IC1, IC5, J1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

Commit message: rough positioning
Parts:
- added D?: D_Schottky, Diodes_SMD:D_SMA, symbol Device:D_Schottky
Connections:
- net VBUS: now also D?.2 (A)
- net VIN: now also D?.1 (K)
Changed lines of the file:
@@
 	18250 2300 18250 900
 Wire Wire Line
-	18250 900  17850 900
+	18250 900  18000 900
 Connection ~ 17850 900
 Connection ~ 18250 900
@@
 Text Notes 21600 9200 0    50   ~ 0
 2X PWM Push-Pull
+Text GLabel 18300 650  2    50   Input ~ 0
+VBUS
+$Comp
+L Device:D_Schottky D?
+U 1 1 60E97C77
+P 18150 650
+F 0 "D?" H 18150 433 50  0000 C CNN
+F 1 "D_Schottky" H 18150 524 50  0000 C CNN
+F 2 "Diodes_SMD:D_SMA" H 18150 650 50  0001 C CNN
+F 3 "~" H 18150 650 50  0001 C CNN
+	1    18150 650
+	1    0    0    -1
+$EndComp
+Wire Wire Line
+	18000 650  18000 900
+Connection ~ 18000 900
+Wire Wire Line
+	18000 900  17850 900
 $EndSCHEMATC
